Commit message: test with donny data

File: urdf/test2.urdf (robot description, URDF)
Before this commit: robot cartographer_my_robot, 5 links, 4 joints
Links:
- removed link frame_velodyne_points
- added link velodyne; visual cylinder length=0.07 radius=0.05
Joints:
- joint velodyne_joint: child frame_velodyne_points -> velodyne; origin xyz=0.04 -0.02 +0.30 rpy=0.0 0.0 0.0 -> xyz=0 0 0 rpy=0.0 0.0 0.0
- joint velodyne_joint_between: parent frame_velodyne_points -> velodyne
